File: Minimal_Prototype_Function_Generator_V0.1/AD9106.kicad_sch (KiCad schematic)
At the start: 30 parts, among them IC1 AD9106BCPZ, J1 142-0701-201, Y1 AX3DCF1-156.2500T

Commit message: Routing PCB, not yet finished
Parts:
- removed TR1: ADT2-1T, RF_Mini-Circuits:Mini-Circuits_CD542_H2.84mm, symbol Transformer:ADT2-1T
- added T1: ADT2-1T+, Insyte_Footprints:ADT21T, symbol ADT2-1T+:ADT2-1T+
Connections:
- net GND: now also T1.3 (PRIMARY_DOT), T1.5 (SECONDARY_CT)
- net at J1.1 (In): now also T1.1 (PRIMARY)
- net at JP1.1 (A): now also T1.4 (SECONDARY)
- net at JP2.3 (B): now also T1.6 (SECONDARY_DOT)
- no-connect marks 0 -> 1
Other:
- moved on the sheet: C6, C7, C8, J1, JP1, JP2, R4, Y1

Commit message: Implemented almost all feedback
Connections:
- net at C8.2, R4.2: now also JP2.3 (B); no longer JP2.1 (A)
- net at T1.6 (SECONDARY_DOT): now also JP2.1 (A); no longer JP2.3 (B)
Changed lines of the file:
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@@
 		(lib_id "Jumper:Jumper_3_Open")
 		(at 95.25 64.77 90)
+		(mirror x)
 		(unit 1)
 		(exclude_from_sim no)
@@
 		(on_board yes)
 		(dnp no)
-		(fields_autoplaced yes)
 		(property "Reference" "JP2"
-			(at 92.71 66.0401 90)
+			(at 92.202 63.5 90)
 			(effects
 				(font
@@
 		)
 		(property "Value" "Jumper_3_Open"
-			(at 92.71 63.5001 90)
+			(at 92.202 66.04 90)
 			(effects
 				(font
