File: Minimal_Prototype_Function_Generator_V0.1/USB_C.kicad_sch (KiCad schematic)
At the start: 8 parts, among them J9 USB4500-03-0-A

Commit message: Routing PCB, not yet finished
Connections:
- net D+: now also D5.2 (K); no longer D5.1 (K)
- net D-: now also D5.1 (K); no longer D5.2 (K)
Changed lines of the file:
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@@
 	)
 	(label "D-"
-		(at 154.94 26.67 180)
+		(at 149.86 26.67 180)
 		(effects
 			(font
@@
 	)
 	(label "D+"
-		(at 149.86 26.67 180)
+		(at 154.94 26.67 180)
 		(effects
 			(font

Commit message: Preliminary delivery of PCB, v0.1
Connections:
- net CC1: now also D4.2 (K); no longer D4.1 (K)
- net CC2: now also D4.1 (K); no longer D4.2 (K)
Changed lines of the file:
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@@
 	)
 	(label "CC2"
-		(at 144.78 26.67 90)
+		(at 139.7 26.67 90)
 		(effects
 			(font
@@
 	)
 	(label "CC1"
-		(at 139.7 26.67 90)
+		(at 144.78 26.67 90)
 		(effects
 			(font

Commit message: Implemented almost all feedback
Other:
- note added: "Impedance calculation for USB4500-03-0-A: (USB2.0 protocol requires 90Ohm diff. impedance and max 0.1mm length discrepancy) JLC impedance calculator for board JLC04161H-7628 (differential pair, non-coplanar) For track spacing 0.2mm, track width is 0.2840mm"
Changed lines of the file:
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@@
+		)
+	)
+	(text "Impedance calculation for USB4500-03-0-A:\n(USB2.0 protocol requires 90Ohm diff. impedance and max 0.1mm length discrepancy)\nJLC impedance calculator for board JLC04161H-7628\n(differential pair, non-coplanar)\nFor track spacing 0.2mm, track width is 0.2840mm"
+		(exclude_from_sim no)
+		(at 61.214 91.948 0)
+		(effects
+			(font
+				(size 1.27 1.27)
+			)
 		)
 	)
