File: Minimal_Prototype_Function_Generator_V0.1/Minimal_Prototype_Function_Generator_V0.1.kicad_pcb (KiCad board)
At the start: 4 copper layers, 9.2 x 6.2 mm, 169 parts, among them IC1 AD9106BCPZ, IC2 ADP5300ACPZ-1-R7, IC3 ADM7160ACPZN3.3-R7, IC4 LT3472EDD#PBF, IC6 ADM7160ACPZN3.3-R7, IC7 ADM7160ACPZN3.3-R7, IC8 ADM7160ACPZN3.3-R7, IC9 STM32L476VGT6, J1 142-0701-201, J10 SPI_TP_1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

Commit message: Routing PCB, not yet finished
Parts:
- removed TR1: ADT2-1T, RF_Mini-Circuits:Mini-Circuits_CD542_H2.84mm
- added T1: ADT2-1T+, Insyte_Footprints:ADT21T, F.Cu at (196.0, 112.0)
- C65, C66: moved to B.Cu
- moved R40 168.7 mm to (57.5, 162.0), turned to -90 degrees
- moved U3 166.7 mm to (63.8, 160.9)
- moved R36 164.2 mm to (56.0, 162.0), turned to -90 degrees
- moved R44 162.2 mm to (62.2, 165.0), turned to 90 degrees
- moved R41 160.7 mm to (66.2, 165.8), turned to 180 degrees
- moved R35 160.5 mm to (59.7, 159.0), turned to 180 degrees
- moved C33 159.3 mm to (78.2, 121.7), turned to 180 degrees
- moved C54 159.1 mm to (59.7, 162.8), turned to 180 degrees
- moved R31 158.9 mm to (56.7, 164.3)
- moved C56 157.3 mm to (60.7, 165.0), turned to 90 degrees
- moved R43 157.2 mm to (66.1, 157.5), turned to 180 degrees
- moved R29 156.5 mm to (58.5, 156.0), turned to 180 degrees
- moved R30 156.3 mm to (58.5, 157.5)
- moved R39 156.0 mm to (61.5, 156.0)
- moved R33 154.4 mm to (69.2, 164.3), turned to 180 degrees
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Connections:
- D5 pad 1: /USB_C/D+ -> /USB_C/D-
- D5 pad 2: /USB_C/D- -> /USB_C/D+
Routing:
- net GND: track 0.00 -> 57.6 mm, vias 0 -> 51
- net /Output_Stage/P5V2: track 0.00 -> 32.8 mm, vias 0 -> 13
- net /Power/LT3472EDD/P5V2_VP: track 0.00 -> 15.3 mm
- net /Power/5V: track 0.00 -> 12.7 mm
- net Net-(IC4-FBN): track 0.00 -> 10.8 mm
- net /Power/VDD_STM32: track 0.00 -> 10.4 mm, vias 0 -> 1
- net /Output_Stage/Op_Amp_1/+IN_2: track 0.00 -> 7.86 mm
- net /Output_Stage/Op_Amp_1/+IN_1: track 0.00 -> 7.44 mm
- net /Output_Stage/Op_Amp_2/+IN_2: track 0.00 -> 7.39 mm
- net /Output_Stage/Op_Amp_2/+IN_1: track 0.00 -> 7.33 mm
- net Net-(IC4-SWN): track 0.00 -> 7.18 mm
- net Net-(IC4-FBP): track 0.00 -> 6.32 mm
- net /Power/ADM7160ACPZN3.3_1/+3V6: track 0.00 -> 6.28 mm
- net Net-(IC9-PC14/OSC32_IN): track 0.00 -> 5.93 mm
- net /Power/LT3472EDD/N5V2_VN: track 0.00 -> 5.77 mm
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- added copper zone on F.Cu, net /Output_Stage/N5V2
- added copper zone on B.Cu, net /Output_Stage/P5V2
- added copper zone on F.Cu, net /Power/VDD_STM32
- added copper zone on B.Cu, net GND
- added copper zone on F.Cu, net GND
- added copper zone on In1.Cu, net GND
- added copper zone on In2.Cu, net GND
Other:
- board size 9.2 x 6.2 mm -> 117.9 x 103.2 mm
- board text added: "Boot pull-down"
- board text added: "Boot pull-up"

Commit message: Preliminary delivery of PCB, v0.1
Parts:
- C19, C20, C21, C22, D4, R51, R52: moved to B.Cu
- moved +3V3_3 151.9 mm to (110.3, 63.1), turned to 180 degrees
- moved +3V3_5 141.6 mm to (109.2, 78.0), turned to 90 degrees
- moved C67 141.5 mm to (115.3, 69.1), turned to 90 degrees
- moved C68 140.5 mm to (115.9, 74.6)
- moved IC8 135.8 mm to (115.9, 72.2), turned to 90 degrees
- moved D1 124.9 mm to (121.6, 58.8), turned to 90 degrees
- moved +5V_1 122.6 mm to (119.8, 52.4)
- moved +3V6_1 119.6 mm to (121.2, 66.0)
- moved R17 119.1 mm to (147.8, 69.5), turned to 180 degrees
- moved L1 119.1 mm to (127.1, 62.4), turned to -90 degrees
- moved R3 116.6 mm to (120.1, 58.8), turned to 90 degrees
- moved R19 116.5 mm to (148.6, 71.8), turned to 90 degrees
- moved C46 115.5 mm to (143.8, 68.8), turned to -90 degrees
- moved R2 115.3 mm to (120.9, 61.0), turned to 180 degrees
- moved C3 114.9 mm to (120.9, 62.5), turned to 180 degrees
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Connections:
- D4 pad 1: /USB_C/CC1 -> /USB_C/CC2
- D4 pad 2: /USB_C/CC2 -> /USB_C/CC1
Routing:
- net /Output_Stage/N5V2: track 0.00 -> 80.8 mm, vias 0 -> 7
- net /USB_C/D-: track 0.00 -> 72.4 mm, vias 0 -> 2
- net /USB_C/D+: track 0.00 -> 72.2 mm, vias 0 -> 2
- net GND: track 57.6 -> 121.5 mm, vias 51 -> 102
- net /Power/ADM7160ACPZN3.3_1/+3V6: track 6.28 -> 70.0 mm, vias 0 -> 2
- net /Output_Stage/Op_Amp_1/AMP1_OUT: track 0.00 -> 60.7 mm, vias 0 -> 3
- net /Output_Stage/Op_Amp_1/AMP_OUT: track 0.00 -> 54.2 mm, vias 0 -> 3
- net /Function Generator/AVDD: track 1.53 -> 54.5 mm, vias 0 -> 2
- net /Output_Stage/P5V2: track 32.8 -> 85.7 mm, vias 13 -> 14
- net Net-(J6-In): track 0.00 -> 45.3 mm, vias 0 -> 2
- net /Power/5V: track 12.7 -> 56.9 mm, vias 0 -> 4
- net /Function Generator/!RESET: track 0.00 -> 34.0 mm, vias 0 -> 2
- net /Function Generator/I_Out_P1: track 1.48 -> 29.5 mm
- net /Function Generator/SPI_CLK: track 0.00 -> 26.5 mm
- net /Function Generator/SPI_MOSI: track 0.00 -> 26.2 mm, vias 0 -> 2
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- added copper zone on F.Cu, net /Power/5V
- added copper zone on F.Cu, net /Power/ADM7160ACPZN3.3_1/+3V6
Other:
- board size 117.9 x 103.2 mm -> 72.3 x 80.6 mm

Commit message: PCB delivery, v1.0
Parts:
- added U4: ~, Insyte_Logo_Footprints:15x6_Insyte_Logo, F.Cu at (60.4, 37.8)
- moved J2 66.7 mm to (58.3, 104.9)
- moved J3 55.6 mm to (79.6, 105.5)
- moved +3V3_5 54.7 mm to (76.2, 34.4)
- moved J4 48.2 mm to (79.6, 91.3)
- moved L1 42.5 mm to (90.5, 40.6), turned to 0 degrees
- moved D5 40.7 mm to (96.2, 49.4)
- moved P5V2_TP1 39.0 mm to (117.9, 34.9)
- moved C19 38.2 mm to (99.6, 71.0)
- moved C20 38.2 mm to (99.6, 69.5)
- moved C21 38.2 mm to (99.6, 72.5)
- moved C22 38.2 mm to (99.6, 74.0)
- moved C36 38.2 mm to (120.0, 69.0)
- moved C38 38.2 mm to (111.1, 54.5)
- moved C39 38.2 mm to (104.7, 50.1)
- moved C41 38.2 mm to (102.8, 56.8)
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Routing:
- net /Output_Stage/Op_Amp_1/AMP_OUT: track 54.2 -> 82.3 mm
- net /Output_Stage/Op_Amp_1/AMP1_OUT: track 60.7 -> 73.8 mm
- net /Output_Stage/Op_Amp_2/AMP_OUT: track 9.73 -> 19.1 mm
- net /Power/VDD_STM32: track 22.4 -> 14.8 mm
- net /USB_C/D-: track 72.4 -> 64.9 mm
- net /USB_C/D+: track 72.2 -> 65.0 mm
- net Net-(J6-In): track 45.3 -> 51.1 mm
- net Net-(IC2-SW): track 7.54 -> 2.40 mm, vias 2 -> 0
- net /Output_Stage/P5V2: track 85.7 -> 90.1 mm, vias 14 -> 15
- net /Output_Stage/Op_Amp_2/AMP1_OUT: track 18.3 -> 21.9 mm
- net /Output_Stage/N5V2: track 80.8 -> 84.0 mm, vias 7 -> 8
- net /USB_C/CC2: track 6.38 -> 9.47 mm
- net /Power/ADM7160ACPZN3.3_1/+3V6: track 70.0 -> 67.6 mm, vias 2 -> 1
- net /Power/5V: track 56.9 -> 55.6 mm, vias 4 -> 3
- net Net-(D1-A): track 7.48 -> 8.46 mm
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Other:
- board text added: "(AVDD)"
- board text added: "(CVVDX)"
- board text added: "(VDD_STM32)"
- board text added: "AMP1"
- board text added: "AMP2"
- board text added: "Amplifier #1 OUTPUT"
- board text added: "Amplifier #1 OUTPUT1"
- board text added: "Amplifier #2 OUTPUT"
- board text added: "Amplifier #2 OUTPUT1"
- board text added: "R49 - boot pull-up"
- board text added: "R50 - boot pull-down"
- board text added: "RF transformer {dblquote}PRIMARY{dblquote} pin"
- board text added: "This PCB is made with love and care"
- board text added: "Trigger input to function generator"
- board text removed: "Boot pull-down"
- board text removed: "Boot pull-up"

Commit message: Implemented almost all feedback
Parts:
- moved JP2 5.08 mm to (108.3, 75.5), turned to 180 degrees
- moved J1 1.85 mm to (110.3, 92.8)
Connections:
- C8 pad 2: Net-(JP2-A) -> Net-(JP2-B)
- R4 pad 2: Net-(JP2-A) -> Net-(JP2-B)
- T1 pad 6: Net-(JP2-B) -> Net-(JP2-A)
Routing:
- net Net-(J6-In): track 51.1 -> 53.5 mm
- net Net-(J1-In): track 7.78 -> 9.62 mm
- net /USB_C/D+: track 65.0 -> 66.3 mm
- net /USB_C/D-: track 64.9 -> 66.1 mm
- net Net-(IC4-FBN): track 10.8 -> 10.1 mm, vias 0 -> 2
- net Net-(JP2-A): track 4.40 -> 3.83 mm
- net Net-(IC4-SWN): track 7.18 -> 7.75 mm
- net GND: vias 306 -> 326
Other:
- board text added: "Debug UART"
- board text added: "Function generator for project EFRO"
- board text added: "I2C_SCL"
- board text added: "I2C_SDA"
- board text added: "JP1 - clock select for {dblquote}SECONDARY{dblquote} winding JP2 - clock select for {dblquote}SECONDARY_DOT{dblquote} winding (pin 2 and 3 are in the same rectangle)"
- board text added: "Output 1 (IOUT1)"
- board text added: "Output 2 (IOUT2)"
- board text added: "Output 3 (IOUT3)"
- board text added: "Output 4 (IOUT4)"
- board text added: "PCB v1.0"
- board text added: "RF transformer External clock supply"
- board text added: "RX"
- board text added: "SPI_CLK"
- board text added: "SPI_CS"
- board text added: "SPI_MISO"
- board text added: "SPI_MOSI"
- board text added: "TX"
- board text removed: "Amplifier #1 OUTPUT"
- board text removed: "Amplifier #1 OUTPUT1"
- board text removed: "Amplifier #2 OUTPUT"
- board text removed: "Amplifier #2 OUTPUT1"
- board text removed: "RF transformer {dblquote}PRIMARY{dblquote} pin"
- board text removed: "This PCB is made with love and care"

Commit message: Ready for order
Other:
- board text added: "Function generator"
- board text removed: "Function generator for project EFRO"
