File: Minimal_Prototype_Function_Generator_V0.1/STM32.kicad_sch (KiCad schematic)
At the start: 24 parts, among them IC9 STM32L476VGT6, J10 SPI_TP_1, J7 DEBUG_UART_TP_1, J8 I2C_TP1, Y2 ECS-.327-7-16-C-TR

Commit message: PCB delivery, v1.0
Parts:
- added U4: ~, Insyte_Logo_Footprints:15x6_Insyte_Logo, symbol Insyte:Logo
Changed lines of the file:
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@@
+	)
+	(symbol
+		(lib_id "Insyte:Logo")
+		(at 194.31 146.05 0)
+		(unit 1)
+		(exclude_from_sim no)
+		(in_bom yes)
+		(on_board yes)
+		(dnp no)
+		(fields_autoplaced yes)
+		(property "Reference" "U4"
+			(at 198.12 144.7799 0)
+			(effects
+				(font
+					(size 1.27 1.27)
+				)
+				(justify left)
+			)
+		)
+		(property "Value" "~"
+			(at 198.12 147.3199 0)
+			(effects
+				(font
+					(size 1.27 1.27)
+				)
+				(justify left)
+			)
+		)
+		(property "Footprint" "Insyte_Logo_Footprints:15x6_Insyte_Logo"
+			(at 194.31 146.05 0)
+			(effects
+				(font
+					(size 1.27 1.27)
+				)
+				(hide yes)
+			)
+		)
+		(property "Datasheet" ""
+			(at 194.31 146.05 0)
+			(effects
+				(font
+					(size 1.27 1.27)
+				)
+				(hide yes)
+			)
+		)
+		(property "Description" ""
+			(at 194.31 146.05 0)
+			(effects
+				(font
+					(size 1.27 1.27)
+				)
+				(hide yes)
+			)
+		)
+		(instances
+			(project ""
+				(path "/4f62c91b-90a7-42e6-9468-9a44c0d5e9c2/41d5001e-a8ed-4e44-9ec1-df5bd6f03dd6"
+					(reference "U4")
+					(unit 1)
+				)
+			)
+		)
 	)
 	(symbol

Commit message: Order
Parts:
- C57, C58, C59, C60, C61, C65: value 0.1u -> 0.1uF
- C62: value 4.7u -> 4.7uF
- C63: value 0.01u -> 0.01uF
- C64, C66: value 1u -> 1uF
- R49, R50: LCSC Part # C23162 -> (none)
Changed lines of the file:
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@@
 			)
 		)
-		(property "Value" "0.1u"
+		(property "Value" "0.1uF"
 			(at 39.624 35.306 0)
 			(effects
@@
 			)
 		)
-		(property "Value" "0.1u"
+		(property "Value" "0.1uF"
 			(at 75.184 35.306 0)
 			(effects
@@
 			)
 		)
-		(property "Value" "4.7u"
+		(property "Value" "4.7uF"
 			(at 96.52 35.306 0)
 			(effects
@@
 			)
 		)
-		(property "Value" "0.1u"
+		(property "Value" "0.1uF"
 			(at 127 35.306 0)
 			(effects
@@
 			)
 		)
-		(property "Value" "0.1u"
+		(property "Value" "0.1uF"
 			(at 63.754 35.306 0)
 			(effects
@@
 			)
 		)
-		(property "Value" "1u"
+		(property "Value" "1uF"
 			(at 116.586 35.052 0)
 			(effects
@@
 			)
 		)
-		(property "Value" "0.1u"
+		(property "Value" "0.1uF"
 			(at 52.324 35.306 0)
 			(effects
@@
 			)
 		)
-		(property "LCSC Part #" " C23162"
+		(property "LCSC Part #" ""
 			(at 97.79 72.39 0)
 			(effects
@@
 			)
 		)
-		(property "Value" "0.1u"
+		(property "Value" "0.1uF"
 			(at 28.194 35.306 0)
 			(effects
@@
 			)
 		)
-		(property "Value" "1u"
+		(property "Value" "1uF"
 			(at 140.716 35.052 0)
 			(effects
@@
 			)
 		)
-		(property "Value" "0.01u"
+		(property "Value" "0.01uF"
 			(at 101.854 35.306 0)
 			(effects
@@
 			)
 		)
-		(property "LCSC Part #" " C23162"
+		(property "LCSC Part #" ""
 			(at 97.79 64.77 0)
 			(effects
